Commit message: Fix duplicate tool0 link error
- Made flange-tool0 joint conditional on use_soft_ee:=false
- Soft EE now connects to flange and creates ee_body-tool0 joint
- Uses existing tool0 link from main xacro

File: ros2_ws/src/mycobot_description/urdf/mech/soft_end_effector.urdf.xacro (robot description, xacro)
@@ -54,9 +54,9 @@
       </collision>
     </link>
-    <!-- Joint from robot to soft tip -->
+    <!-- Joint from robot flange to soft tip -->
+    <!-- Connects to flange instead of wrist_3_link to avoid duplicate tool0 -->
     <joint name="${prefix}ee_mount" type="fixed">
       <parent link="${parent_link}"/>
       <child link="${prefix}soft_tip"/>
-      <!-- Adjust this offset to position your EE correctly -->
       <origin xyz="0 0 0" rpy="0 0 0"/>
     </joint>
@@ -67,11 +67,10 @@
       <origin xyz="0 0 0" rpy="0 0 0"/>
     </joint>
-    <!-- TOOL FRAME - Required for MoveIt! -->
-    <!-- Position this at the tip of your end effector -->
-    <link name="${prefix}tool0"/>
-    <joint name="${prefix}tool0_joint" type="fixed">
+    <!-- TOOL FRAME - Connect existing tool0 to end of EE -->
+    <!-- The tool0 link is already defined in main xacro, we just connect it to our EE -->
+    <joint name="${prefix}ee_body-tool0" type="fixed">
       <parent link="${prefix}ee_body"/>
       <child link="${prefix}tool0"/>
-      <!-- Adjust based on your EE geometry - currently at body center -->
+      <!-- Position at tip of end effector - ADJUST THIS VALUE -->
       <origin xyz="0 0 0.06" rpy="0 0 0"/>
     </joint>

File: ros2_ws/src/mycobot_description/urdf/robots/mycobot_320_ur_compatible.urdf.xacro (robot description, xacro)
@@ -244,10 +244,12 @@
       <origin xyz="0 0 0" rpy="0 ${-pi/2.0} ${-pi/2.0}"/>
     </joint>
-    <!-- flange-tool0 fixed joint -->
-    <joint name="$(arg prefix)flange-tool0" type="fixed">
-      <parent link="$(arg prefix)flange"/>
-      <child link="$(arg prefix)tool0"/>
-      <origin xyz="0 0 0" rpy="0 0 0"/>
-    </joint>
+    <!-- flange-tool0 fixed joint - Only add if NOT using soft end effector -->
+    <xacro:unless value="$(arg use_soft_ee)">
+      <joint name="$(arg prefix)flange-tool0" type="fixed">
+        <parent link="$(arg prefix)flange"/>
+        <child link="$(arg prefix)tool0"/>
+        <origin xyz="0 0 0" rpy="0 0 0"/>
+      </joint>
+    </xacro:unless>
     <!-- Gazebo Sim ROS2 Control Plugin -->
     <xacro:include filename="$(find mycobot_description)/urdf/control/gazebo_sim_ros2_control.urdf.xacro"/>
@@ -260,5 +262,5 @@
     <!-- Conditionally add soft end effector -->
     <xacro:if value="$(arg use_soft_ee)">
-      <xacro:soft_end_effector parent_link="$(arg prefix)wrist_3_link" prefix="$(arg prefix)"/>
+      <xacro:soft_end_effector parent_link="$(arg prefix)flange" prefix="$(arg prefix)"/>
     </xacro:if>
     <!-- UR-compatible ROS2 Control Configuration -->
